File: KiCad/CH552E2x2.kicad_sch (KiCad schematic)
At the start: 21 parts, among them J1 USB_C_Receptacle_USB2.0, SW1 Switch, U1 CH552E, U2 PRTR5V0U2X

Commit message: Update
Solder -> Hot Swap
THT -> SMD Diodes
Screw Hole -> Not Inconvenient Anymore
Parts:
- D3, D4, D5, D6: footprint VyPrints:D_DO-35_SOD27_P7.62mm_Horizontal -> Diode_SMD:D_SOD-123
- MX1: footprint PCM_marbastlib-mx:SW_MX_1u -> PCM_marbastlib-mx:SW_MX_HS_CPG151101S11_1u
Changed lines of the file:
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@@
 				)
 			)
-			(project "CH552ETEST"
+			(project "CH552E2x2"
 				(path "/ac567297-42ff-4d14-a5ad-ac820d24b8fa"
 					(reference "#PWR03")
@@
 			)
 		)
-		(property "Footprint" "VyPrints:D_DO-35_SOD27_P7.62mm_Horizontal"
+		(property "Footprint" "Diode_SMD:D_SOD-123"
 			(at 125.095 85.09 0)
 			(effects
@@
 		)
 		(instances
-			(project "CH552ETEST"
+			(project "CH552E2x2"
 				(path "/ac567297-42ff-4d14-a5ad-ac820d24b8fa"
 					(reference "D5")
@@
 				)
 			)
-			(project "CH552ETEST"
+			(project "CH552E2x2"
 				(path "/ac567297-42ff-4d14-a5ad-ac820d24b8fa"
 					(reference "#PWR08")
@@
 				)
 			)
-			(project "CH552ETEST"
+			(project "CH552E2x2"
 				(path "/ac567297-42ff-4d14-a5ad-ac820d24b8fa"
 					(reference "F1")
@@
 				)
 			)
-			(project "CH552ETEST"
+			(project "CH552E2x2"
 				(path "/ac567297-42ff-4d14-a5ad-ac820d24b8fa"
 					(reference "#PWR02")
@@
 				)
 			)
-			(project "CH552ETEST"
+			(project "CH552E2x2"
 				(path "/ac567297-42ff-4d14-a5ad-ac820d24b8fa"
 					(reference "C2")
@@
 				)
 			)
-			(project "CH552ETEST"
+			(project "CH552E2x2"
 				(path "/ac567297-42ff-4d14-a5ad-ac820d24b8fa"
 					(reference "#PWR012")
@@
 			)
 		)
-		(property "Footprint" "VyPrints:D_DO-35_SOD27_P7.62mm_Horizontal"
+		(property "Footprint" "Diode_SMD:D_SOD-123"
 			(at 141.605 62.23 0)
 			(effects
@@
 		)
 		(instances
-			(project "CH552ETEST"
+			(project "CH552E2x2"
 				(path "/ac567297-42ff-4d14-a5ad-ac820d24b8fa"
 					(reference "D4")
@@
 				)
 			)
-			(project "CH552ETEST"
+			(project "CH552E2x2"
 				(path "/ac567297-42ff-4d14-a5ad-ac820d24b8fa"
 					(reference "#PWR04")
@@
 			)
 		)
-		(property "Footprint" "VyPrints:D_DO-35_SOD27_P7.62mm_Horizontal"
+		(property "Footprint" "Diode_SMD:D_SOD-123"
 			(at 138.43 85.09 0)
 			(effects
@@
 		)
 		(instances
-			(project "CH552ETEST"
+			(project "CH552E2x2"
 				(path "/ac567297-42ff-4d14-a5ad-ac820d24b8fa"
 					(reference "D6")
@@
 				)
 			)
-			(project "CH552ETEST"
+			(project "CH552E2x2"
 				(path "/ac567297-42ff-4d14-a5ad-ac820d24b8fa"
 					(reference "R2")
@@
 		)
 		(instances
-			(project "CH552ETEST"
+			(project "CH552E2x2"
 				(path "/ac567297-42ff-4d14-a5ad-ac820d24b8fa"
 					(reference "#PWR015")
@@
 				)
 			)
-			(project "CH552ETEST"
+			(project "CH552E2x2"
 				(path "/ac567297-42ff-4d14-a5ad-ac820d24b8fa"
 					(reference "RESET1")
@@
 				)
 			)
-			(project "CH552ETEST"
+			(project "CH552E2x2"
 				(path "/ac567297-42ff-4d14-a5ad-ac820d24b8fa"
 					(reference "R1")
@@
 				)
 			)
-			(project "CH552ETEST"
+			(project "CH552E2x2"
 				(path "/ac567297-42ff-4d14-a5ad-ac820d24b8fa"
 					(reference "R4")
@@
 				)
 			)
-			(project "CH552ETEST"
+			(project "CH552E2x2"
 				(path "/ac567297-42ff-4d14-a5ad-ac820d24b8fa"
 					(reference "J1")
@@
 		)
 		(instances
-			(project "CH552ETEST"
+			(project "CH552E2x2"
 				(path "/ac567297-42ff-4d14-a5ad-ac820d24b8fa"
 					(reference "H1")
@@
 				)
 			)
-			(project "CH552ETEST"
+			(project "CH552E2x2"
 				(path "/ac567297-42ff-4d14-a5ad-ac820d24b8fa"
 					(reference "#PWR013")
@@
 				)
 			)
-			(project "CH552ETEST"
+			(project "CH552E2x2"
 				(path "/ac567297-42ff-4d14-a5ad-ac820d24b8fa"
 					(reference "C1")
@@
 			)
 		)
-		(property "Footprint" "PCM_marbastlib-mx:SW_MX_1u"
+		(property "Footprint" "PCM_marbastlib-mx:SW_MX_HS_CPG151101S11_1u"
 			(at 113.665 55.245 0)
 			(effects
@@
 				)
 			)
-			(project "CH552ETEST"
+			(project "CH552E2x2"
 				(path "/ac567297-42ff-4d14-a5ad-ac820d24b8fa"
 					(reference "MX1")
@@
 			)
 		)
-		(property "Footprint" "PCM_marbastlib-mx:SW_MX_1u"
+		(property "Footprint" "PCM_marbastlib-mx:SW_MX_HS_CPG151101S11_1u"
 			(at 127 55.245 0)
 			(effects
@@
 				)
 			)
-			(project "CH552ETEST"
+			(project "CH552E2x2"
 				(path "/ac567297-42ff-4d14-a5ad-ac820d24b8fa"
 					(reference "MX2")
@@
 				)
 			)
-			(project "CH552ETEST"
+			(project "CH552E2x2"
 				(path "/ac567297-42ff-4d14-a5ad-ac820d24b8fa"
 					(reference "BOOT1")
@@
 				)
 			)
-			(project "CH552ETEST"
+			(project "CH552E2x2"
 				(path "/ac567297-42ff-4d14-a5ad-ac820d24b8fa"
 					(reference "U1")
@@
 			)
 		)
-		(property "Footprint" "PCM_marbastlib-mx:SW_MX_1u"
+		(property "Footprint" "PCM_marbastlib-mx:SW_MX_HS_CPG151101S11_1u"
 			(at 123.825 78.105 0)
 			(effects
@@
 				)
 			)
-			(project "CH552ETEST"
+			(project "CH552E2x2"
 				(path "/ac567297-42ff-4d14-a5ad-ac820d24b8fa"
 					(reference "MX4")
@@
 			)
 		)
-		(property "Footprint" "PCM_marbastlib-mx:SW_MX_1u"
+		(property "Footprint" "PCM_marbastlib-mx:SW_MX_HS_CPG151101S11_1u"
 			(at 110.49 78.105 0)
 			(effects
@@
 				)
 			)
-			(project "CH552ETEST"
+			(project "CH552E2x2"
 				(path "/ac567297-42ff-4d14-a5ad-ac820d24b8fa"
 					(reference "MX3")
@@
 				)
 			)
-			(project "CH552ETEST"
+			(project "CH552E2x2"
 				(path "/ac567297-42ff-4d14-a5ad-ac820d24b8fa"
 					(reference "D1")
@@
 				)
 			)
-			(project "CH552ETEST"
+			(project "CH552E2x2"
 				(path "/ac567297-42ff-4d14-a5ad-ac820d24b8fa"
 					(reference "#PWR011")
@@
 				)
 			)
-			(project "CH552ETEST"
+			(project "CH552E2x2"
 				(path "/ac567297-42ff-4d14-a5ad-ac820d24b8fa"
 					(reference "#PWR05")
@@
 		)
 		(instances
-			(project "CH552ETEST"
+			(project "CH552E2x2"
 				(path "/ac567297-42ff-4d14-a5ad-ac820d24b8fa"
 					(reference "U2")
@@
 				)
 			)
-			(project "CH552ETEST"
+			(project "CH552E2x2"
 				(path "/ac567297-42ff-4d14-a5ad-ac820d24b8fa"
 					(reference "#PWR06")
@@
 			)
 		)
-		(property "Footprint" "VyPrints:D_DO-35_SOD27_P7.62mm_Horizontal"
+		(property "Footprint" "Diode_SMD:D_SOD-123"
 			(at 128.27 62.23 0)
 			(effects
@@
 		)
 		(instances
-			(project "CH552ETEST"
+			(project "CH552E2x2"
 				(path "/ac567297-42ff-4d14-a5ad-ac820d24b8fa"
 					(reference "D3")
@@
 				)
 			)
-			(project "CH552ETEST"
+			(project "CH552E2x2"
 				(path "/ac567297-42ff-4d14-a5ad-ac820d24b8fa"
 					(reference "#PWR09")
@@
 				)
 			)
-			(project "CH552ETEST"
+			(project "CH552E2x2"
 				(path "/ac567297-42ff-4d14-a5ad-ac820d24b8fa"
 					(reference "#PWR010")
